Commit message: ackermann urdf

File: clu_description/urdf/ackermann_rover.urdf (robot description, URDF)
Before this commit: robot rover, 6 links, 5 joints
Links:
- added link left_steering_column; visual cyclinder length=0.1 radius=0.01
- added link right_steering_column; visual cyclinder length=0.1 radius=0.01
Joints:
- added joint left_wheel_steering_column: type revolute, parent left_steering_column, child left_wheel, origin xyz=0 0.2 0 rpy=1.57 0 0, axis 1 0 0, limit lower=0.0 upper=0.548 effort=1000.0 velocity=0.5
- added joint right_wheel_steering_column: type revolute, parent right_steering_column, child right_wheel, origin xyz=0 -0.2 0 rpy=1.57 0 0, axis 1 0 0, limit lower=0.0 upper=0.548 effort=1000.0 velocity=0.5
- joint base_left_wheel: child left_wheel -> left_steering_column; origin xyz=0 0.2 0 rpy=1.57 0 0 -> (none)
- joint base_right_wheel: child right_wheel -> right_steering_cloumn; origin xyz=0 -0.2 0 rpy=1.57 0 0 -> (none)
