Commit message: xacro added

File: clu_description/urdf/ackermann_rover.xacro (robot description, xacro)
@@ -1,4 +1,4 @@
 <?xml version="1.0"?>
-<robot name="ackermann_rover">
+<robot name="ackermann_rover" xmlns:xacro="http://www.ros.org/wiki/xacro">
     <material name="grey">
         <color rgba="0.7 0.7 0.7 1" />
@@ -8,5 +8,5 @@
     </material>
     <material name="blue">
-        <color rgba="1 1 1 1" />
+        <color rgba="0 0 1 1" />
     </material>
     <link name="base_link">
@@ -37,13 +37,4 @@
         </visual>
     </link>
-    <link name="right_steering_column" >
-        <visual>
-            <geometry>
-                <cyclinder radius="0.01" length="0.1" />
-            </geometry>
-            <origin xyz="0 0 0" rpy="0 0 0" />
-            <material name="blue" />
-        </visual>
-    </link>
     <link name="left_wheel">
         <visual>
@@ -55,8 +46,17 @@
         </visual>
     </link>
-    <link name="left_steering_column" >
+    <link name="right_steering_column">
         <visual>
             <geometry>
-                <cyclinder radius="0.01" length="0.1" />
+                <cylinder radius="0.01" length="0.1" />
+            </geometry>
+            <origin xyz="0 0 0" rpy="0 0 0" />
+            <material name="blue" />
+        </visual>
+    </link>
+    <link name="left_steering_column">
+        <visual>
+            <geometry>
+                <cylinder radius="0.01" length="0.1" />
             </geometry>
             <origin xyz="0 0 0" rpy="0 0 0" />
@@ -73,6 +73,5 @@
         </visual>
     </link>
-    <link name="base_footprint">
-    </link>
+    <link name="base_footprint" />
     <joint name="base_lidar_joint" type="fixed">
         <parent link="base_link" />
@@ -80,9 +79,9 @@
         <origin xyz="0 0 0.2" rpy="0 0 0" />
     </joint>
-    <joint name="base_left_wheel" type="continuous" >
+    <joint name="base_left_wheel" type="continuous">
         <parent link="base_link" />
         <child link="left_steering_column" />
-        <axis xyz="1 0 0" rpy="0 0 0" />
-        <axis xyz="0 0 0" />
+        <origin xyz="0 0.2 0" rpy="0 0 0" />
+        <axis xyz="1 0 0" />
     </joint>
     <joint name="left_wheel_steering_column" type="revolute">
@@ -93,5 +92,5 @@
         <limit lower="0.0" upper="0.548" effort="1000" velocity="0.5"/>
     </joint>
-    <joint name="base_right_wheel" type="continuous" >
+    <joint name="base_right_wheel" type="continuous">
         <parent link="base_link" />
         <child link="right_steering_column" />
@@ -109,10 +108,10 @@
         <parent link="base_link" />
         <child link="castor" />
-        <axis xyz="0.15 0 0" rpy="0 0 0" />
+        <origin xyz="0.15 0 0" rpy="0 0 0" />
     </joint>
     <joint name="base_footprint_base_link" type="fixed">
         <parent link="base_footprint" />
         <child link="base_link" />
-        <axis xyz="0 0 0.1" rpy="0 0 0" />
+        <origin xyz="0 0 0.1" rpy="0 0 0" />
     </joint>
 </robot>
